File: PowerSupplyMonitorHub/PowerSupplyMonitorHub.kicad_pcb (KiCad board)
At the start: 2 copper layers, 145 x 62 mm, 90 parts, among them J1 CON_PCA, J10 Input, J2 RJ45 PWR 0, J3 RJ45 PWR 1, J4 RJ45 PWR 2, J5 RJ45 PWR 3, J6 RJ45 PWR 4, J7 OLED I2C, J8 CON_TCA, J9 CON_PCF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

Commit message: added small changes to power supply pcbs added needed libraries to node firmware folder added node test program for wemos D1 mini as master added placeholder header and source file for new firmware
Routing:
- net GND: track 0.00 -> 6.06 mm, vias 77 -> 104
- net /DC-OK_1: track 20.1 -> 24.0 mm
- net /DATA_4: track 169.5 -> 171.8 mm
- net /LINK_3: track 111.8 -> 113.9 mm
- net /LINK_0: track 42.9 -> 45.0 mm
- net /LINK_4: track 146.1 -> 147.5 mm
- net /RC_3: track 53.7 -> 54.0 mm, vias 0 -> 1
- net (no net): vias 1 -> 0
