File: PowerSupplyMonitorHub/PowerSupplyMonitorHub.sch (KiCad schematic (older format))
At the start: 89 parts, among them J1 Input, J10 RJ45 PWR 4, J2 OLED I2C, J3 CON_PCA, J4 RJ45 PWR 0, J5 CON_PCF, J6 RJ45 PWR 1, J7 RJ45 PWR 2, J8 CON_TCA, J9 RJ45 PWR 3, SW1 DIP_PCA, SW2 DIP_PCF, SW3 DIP_TCA, U1 PCA9685PW, U10 PC817, U11 PC817, U12 PC817, U13 PC817, U2 PCF8575, U3 PC817, U4 PC817, U5 PC817, U6 PC817, U7 PC817, U8 PC817, U9 TCA9548APWR

Commit message: added dip switches to i2c ics for adress selection added pullup resistors to i2c input lines added placeholder footprint for pcf8575 added minimal pcb placement for testing
Parts:
- U2: footprint IPC7351-Nominal:SOP65P775X200-24 -> Package_SO:SSOP-24_5.3x8.2mm_P0.65mm
- renumbered DS2 to DS1, DS9 to DS10, DS1 to DS2, DS4 to DS3, DS3 to DS4, DS6 to DS5, DS5 to DS6, DS8 to DS7, DS7 to DS8, DS10 to DS9, R37 to R36, R36 to R37, R42 to R40, R40 to R42, R46 to R44, R44 to R46, R48 to R47, R47 to R48, R50 to R49, R49 to R50

Commit message: changed package and footprint from sop to soi for pcf8575
Parts:
- U2: footprint Package_SO:SSOP-24_5.3x8.2mm_P0.65mm -> Package_SO:SOIC-24W_7.5x15.4mm_P1.27mm
Changed lines of the file:
@@
 F 0 "U2" V 3896 3670 50  0000 R CNN
 F 1 "PCF8575" V 3805 3670 50  0000 R CNN
-F 2 "Package_SO:SSOP-24_5.3x8.2mm_P0.65mm" H 3850 3600 50  0001 C CNN
+F 2 "Package_SO:SOIC-24W_7.5x15.4mm_P1.27mm" H 3850 3600 50  0001 C CNN
 F 3 "http://www.nxp.com/documents/data_sheet/PCF8575.pdf" H 3850 3500 50  0001 C CNN
 F 4 "NXP" H 3850 3300 50  0001 C CNN "Manuf"

Commit message: added new 3d render of front and back view of pcb added pcb routing from autorouter added power led indicator added i2c ic adress ranges to silkscreen added unused ic pins pinout info silkscreen added power input info silkscreen
Parts:
- added DS11: PWR, LED_SMD:LED_0805_2012Metric_Pad1.15x1.40mm_HandSolder, symbol _semi:LED
- added MH1, MH2, MH3, MH4: MountingHole, MountingHole:MountingHole_3.5mm, symbol Mechanical:MountingHole
- added R51: 220, Resistor_SMD:R_0805_2012Metric_Pad1.15x1.40mm_HandSolder, symbol Device:R
- renumbered J3 to J1, J1 to J10, J4 to J2, J6 to J3, J7 to J4, J9 to J5, J10 to J6, J2 to J7, J5 to J9, R13 to R1, R45 to R10, R14 to R11, R19 to R12, R24 to R13, R33 to R14, R41 to R15, R3 to R16, R4 to R17, R5 to R18, R6 to R19, R16 to R2, R7 to R20, R12 to R21, R15 to R22, R17 to R23, R20 to R24, R22 to R25, R28 to R27, R34 to R28, R38 to R29, R18 to R3, R43 to R30, R8 to R31, R1 to R32, R2 to R33, R30 to R34, R25 to R35, R31 to R36, R32 to R37, R36 to R38, R37 to R39, R21 to R4, R42 to R41, R44 to R42, R46 to R43, R47 to R44, R48 to R45, R49 to R46, R50 to R47, R9 to R48, R10 to R49, R23 to R5, R11 to R50, R27 to R6, R29 to R7, R35 to R8, R39 to R9, SW3 to SW2, SW2 to SW3, U12 to U10, U13 to U11, U9 to U12, U2 to U13, U3 to U2, U4 to U3, U5 to U4, U6 to U5, U7 to U6, U8 to U7, U10 to U8, U11 to U9
Connections:
- wire segments 304 -> 294

Commit message: added minimal readme
added many vias for ground front and back plane
updated 3d render of i2c hub pcb
updated gerber archive files
Connections:
- no-connect marks 0 -> 1
Changed lines of the file:
@@
 	1    0    0    -1
 $EndComp
+NoConn ~ 4750 5800
 Wire Bus Line
 	1450 3350 1950 3350

Commit message: updated readme and license file
added datasheet for ads1015
added datasheet for pca9685
added foto of gy-712 30a sensor
added small changes to pcbs
updated 3d render of pcbs
Parts:
- C1: value C_PCA -> 0.1uF
- C2: value C_PCF -> 0.1uF
- C3: value C_TCA -> 0.1uF
Changed lines of the file:
@@
 P 2750 5450
 F 0 "C1" V 2700 5300 50  0000 C CNN
-F 1 "C_PCA" V 2750 5750 50  0000 C CNN
+F 1 "0.1uF" V 2750 5750 50  0000 C CNN
 F 2 "Capacitor_SMD:C_0805_2012Metric_Pad1.15x1.40mm_HandSolder" H 2750 5450 50  0001 C CNN
 F 3 "~" H 2750 5450 50  0001 C CNN
@@
 P 2750 5600
 F 0 "C2" V 2800 5750 50  0000 C CNN
-F 1 "C_PCF" V 2750 5300 50  0000 C CNN
+F 1 "0.1uF" V 2750 5300 50  0000 C CNN
 F 2 "Capacitor_SMD:C_0805_2012Metric_Pad1.15x1.40mm_HandSolder" H 2750 5600 50  0001 C CNN
 F 3 "~" H 2750 5600 50  0001 C CNN
@@
 P 2750 5750
 F 0 "C3" V 2800 5900 50  0000 C CNN
-F 1 "C_TCA" V 2750 5450 50  0000 C CNN
+F 1 "0.1uF" V 2750 5450 50  0000 C CNN
 F 2 "Capacitor_SMD:C_0805_2012Metric_Pad1.15x1.40mm_HandSolder" H 2750 5750 50  0001 C CNN
 F 3 "~" H 2750 5750 50  0001 C CNN

Commit message: fixed pcb errors
swapped gnd and vcc pin of 4 position switch to fix first two addresses
added custom 3d model for 4 position switch as step file
added custom library for 4 position switch
fixed routing of feedback signal lines (dc0-dc5)
removed double current limiting led resistors
Parts:
- removed R22, R24, R26, R28, R30: 220, Resistor_SMD:R_0805_2012Metric_Pad1.15x1.40mm_HandSolder, symbol Device:R
Connections:
- wire segments 294 -> 289
Changed lines of the file:
@@
 Entry Wire Line
 	4700 4100 4800 4200
-$Comp
-L Device:R R22
-U 1 1 5B62100B
-P 4450 3550
-F 0 "R22" V 4550 3450 50  0000 L CNN
-F 1 "220" V 4450 3450 50  0000 L CNN
-F 2 "Resistor_SMD:R_0805_2012Metric_Pad1.15x1.40mm_HandSolder" V 4380 3550 50  0001 C CNN
-F 3 "~" H 4450 3550 50  0001 C CNN
-	1    4450 3550
-	1    0    0    -1
-$EndComp
-Entry Wire Line
-	4350 3900 4450 4000
+Entry Wire Line
+	4450 3900 4550 4000
 Entry Wire Line
 	4050 3900 4150 4000
@@
 Entry Wire Line
 	5900 4100 6000 4200
-$Comp
-L Device:R R24
-U 1 1 5B63D915
-P 5650 3550
-F 0 "R24" V 5750 3450 50  0000 L CNN
-F 1 "220" V 5650 3450 50  0000 L CNN
-F 2 "Resistor_SMD:R_0805_2012Metric_Pad1.15x1.40mm_HandSolder" V 5580 3550 50  0001 C CNN
-F 3 "~" H 5650 3550 50  0001 C CNN
-	1    5650 3550
-	1    0    0    -1
-$EndComp
-Entry Wire Line
-	5550 3900 5650 4000
+Entry Wire Line
+	5650 3900 5750 4000
 Entry Wire Line
 	5250 3900 5350 4000
@@
 Entry Wire Line
 	7100 4100 7200 4200
-$Comp
-L Device:R R26
-U 1 1 5B64175B
-P 6850 3550
-F 0 "R26" V 6950 3450 50  0000 L CNN
-F 1 "220" V 6850 3450 50  0000 L CNN
-F 2 "Resistor_SMD:R_0805_2012Metric_Pad1.15x1.40mm_HandSolder" V 6780 3550 50  0001 C CNN
-F 3 "~" H 6850 3550 50  0001 C CNN
-	1    6850 3550
-	1    0    0    -1
-$EndComp
-Entry Wire Line
-	6750 3900 6850 4000
+Entry Wire Line
+	6850 3900 6950 4000
 Entry Wire Line
 	6450 3900 6550 4000
@@
 	1    0    0    -1
 $EndComp
-$Comp
-L Device:R R28
-U 1 1 5B64CAE6
-P 8050 3550
-F 0 "R28" V 8150 3450 50  0000 L CNN
-F 1 "220" V 8050 3450 50  0000 L CNN
-F 2 "Resistor_SMD:R_0805_2012Metric_Pad1.15x1.40mm_HandSolder" V 7980 3550 50  0001 C CNN
-F 3 "~" H 8050 3550 50  0001 C CNN
-	1    8050 3550
-	1    0    0    -1
-$EndComp
-Entry Wire Line
-	7950 3900 8050 4000
+Entry Wire Line
+	8050 3900 8150 4000
 Entry Wire Line
 	7650 3900 7750 4000
@@
 	1    0    0    -1
 $EndComp
-$Comp
-L Device:R R30
-U 1 1 5B652E68
-P 9250 3550
-F 0 "R30" V 9350 3450 50  0000 L CNN
-F 1 "220" V 9250 3450 50  0000 L CNN
-F 2 "Resistor_SMD:R_0805_2012Metric_Pad1.15x1.40mm_HandSolder" V 9180 3550 50  0001 C CNN
-F 3 "~" H 9250 3550 50  0001 C CNN
-	1    9250 3550
-	1    0    0    -1
-$EndComp
-Entry Wire Line
-	9150 3900 9250 4000
+Entry Wire Line
+	9250 3900 9350 4000
 Entry Wire Line
 	8850 3900 8950 4000
@@
 Text Label 4050 3650 3    50   ~ 0
 RC_0
-Text Label 4350 3650 3    50   ~ 0
+Text Label 4450 3650 3    50   ~ 0
 DC_0
 Text Label 5250 3650 3    50   ~ 0
 RC_1
-Text Label 5550 3650 3    50   ~ 0
+Text Label 5650 3650 3    50   ~ 0
 DC_1
 Text Label 6450 3650 3    50   ~ 0
 RC_2
-Text Label 6750 3650 3    50   ~ 0
+Text Label 6850 3650 3    50   ~ 0
 DC_2
-Text Label 7950 3650 3    50   ~ 0
+Text Label 8050 3650 3    50   ~ 0
 DC_3
 Text Label 7650 3650 3    50   ~ 0
@@
 Text Label 8850 3650 3    50   ~ 0
 RC_4
-Text Label 9150 3650 3    50   ~ 0
+Text Label 9250 3650 3    50   ~ 0
 DC_4
 Text Label 3950 4600 3    50   ~ 0
@@
 	1    0    0    -1
 $EndComp
-Wire Wire Line
-	4350 3900 4350 3400
-Wire Wire Line
-	5550 3900 5550 3400
-Wire Wire Line
-	6750 3900 6750 3400
-Wire Wire Line
-	9150 3400 9150 3900
 Text Label 9300 800  0    50   ~ 0
 LINK_4
@@
 $EndComp
 $Comp
-L power:+5V #PWR032
-U 1 1 5B5FB505
-P 4450 3700
-F 0 "#PWR032" H 4450 3550 50  0001 C CNN
-F 1 "+5V" H 4465 3873 50  0000 C CNN
-F 2 "" H 4450 3700 50  0001 C CNN
-F 3 "" H 4450 3700 50  0001 C CNN
-	1    4450 3700
-	-1   0    0    1
-$EndComp
-$Comp
 L power:+5V #PWR039
 U 1 1 5B5FB56A
@@
 $EndComp
 $Comp
-L power:+5V #PWR033
-U 1 1 5B5FB5CF
-P 5650 3700
-F 0 "#PWR033" H 5650 3550 50  0001 C CNN
-F 1 "+5V" H 5665 3873 50  0000 C CNN
-F 2 "" H 5650 3700 50  0001 C CNN
-F 3 "" H 5650 3700 50  0001 C CNN
-	1    5650 3700
-	-1   0    0    1
-$EndComp
-$Comp
 L power:+5V #PWR041
 U 1 1 5B5FB690
@@
 $EndComp
 $Comp
-L power:+5V #PWR034
-U 1 1 5B5FB6F5
-P 6850 3700
-F 0 "#PWR034" H 6850 3550 50  0001 C CNN
-F 1 "+5V" H 6865 3873 50  0000 C CNN
-F 2 "" H 6850 3700 50  0001 C CNN
-F 3 "" H 6850 3700 50  0001 C CNN
-	1    6850 3700
-	-1   0    0    1
-$EndComp
-$Comp
 L power:+5V #PWR043
 U 1 1 5B5FB7B6
@@
 $EndComp
 $Comp
-L power:+5V #PWR035
-U 1 1 5B5FB81B
-P 8050 3700
-F 0 "#PWR035" H 8050 3550 50  0001 C CNN
-F 1 "+5V" H 8065 3873 50  0000 C CNN
-F 2 "" H 8050 3700 50  0001 C CNN
-F 3 "" H 8050 3700 50  0001 C CNN
-	1    8050 3700
-	-1   0    0    1
-$EndComp
-$Comp
 L power:+5V #PWR045
 U 1 1 5B5FBB52
@@
 F 3 "" H 8650 3700 50  0001 C CNN
 	1    8650 3700
-	-1   0    0    1
-$EndComp
-$Comp
-L power:+5V #PWR036
-U 1 1 5B5FBBB7
-P 9250 3700
-F 0 "#PWR036" H 9250 3550 50  0001 C CNN
-F 1 "+5V" H 9265 3873 50  0000 C CNN
-F 2 "" H 9250 3700 50  0001 C CNN
-F 3 "" H 9250 3700 50  0001 C CNN
-	1    9250 3700
 	-1   0    0    1
 $EndComp
@@
 	0    1    1    0
 $EndComp
-Wire Wire Line
-	9150 3400 9050 3400
-Connection ~ 9050 3400
-Wire Wire Line
-	7950 3900 7950 3400
-Wire Wire Line
-	7850 3400 7950 3400
-Connection ~ 7850 3400
 $Comp
 L power:GND #PWR042
@@
 	1    0    0    -1
 $EndComp
-Wire Wire Line
-	6650 3400 6750 3400
-Connection ~ 6650 3400
-Wire Wire Line
-	5450 3400 5550 3400
-Wire Wire Line
-	4250 3400 4350 3400
 $Comp
 L power:GND #PWR040
@@
 	1    0    0    -1
 $EndComp
-Connection ~ 5450 3400
 $Comp
 L power:GND #PWR038
@@
 	1    0    0    -1
 $EndComp
-Connection ~ 4250 3400
 $Comp
 L Mechanical:MountingHole MH1
@@
 $EndComp
 NoConn ~ 4750 5800
+Wire Wire Line
+	4450 3900 4450 3400
+Wire Wire Line
+	9250 3900 9250 3400
+Wire Wire Line
+	8050 3900 8050 3400
+Wire Wire Line
+	6850 3900 6850 3400
+Wire Wire Line
+	5650 3900 5650 3400
 Wire Bus Line
 	1450 3350 1950 3350
